File: PCBs/KiCad/Wand Board ESP32/Wand Board ESP32.kicad_pcb (KiCad board)
At the start: 2 copper layers, 86 x 56 mm, 28 parts, among them J10 ENC BTN, J11 ENCODER, J12 POW_IN, J13 BRL SENSE, J14 BAR, J15 DISP, J16 BODY LEDS, J17 VIBR, J19 BRL LEDS, J3 TIP LED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

Commit message: Tweaks to jigs, coloured schematics, readme notes
Parts:
- renumbered EC3Z1 to ESP32-C3-Zero1
Changed lines of the file:
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@@
 	(net 12 "/MOT-")
 	(net 13 "Net-(Q1-B)")
-	(net 14 "Net-(EC3Z1-GP8)")
-	(net 15 "Net-(EC3Z1-GP5)")
-	(net 16 "Net-(EC3Z1-GP3)")
-	(net 17 "Net-(EC3Z1-GP2)")
-	(net 18 "Net-(EC3Z1-GP18)")
-	(net 19 "Net-(EC3Z1-GP9)")
-	(net 20 "Net-(EC3Z1-GP6)")
-	(net 21 "Net-(EC3Z1-GP10)")
-	(net 22 "Net-(EC3Z1-GP4)")
-	(net 23 "Net-(EC3Z1-GP19)")
-	(net 24 "Net-(EC3Z1-GP7)")
+	(net 14 "Net-(ESP32-C3-Zero1-GP8)")
+	(net 15 "Net-(ESP32-C3-Zero1-GP5)")
+	(net 16 "Net-(ESP32-C3-Zero1-GP3)")
+	(net 17 "Net-(ESP32-C3-Zero1-GP2)")
+	(net 18 "Net-(ESP32-C3-Zero1-GP18)")
+	(net 19 "Net-(ESP32-C3-Zero1-GP9)")
+	(net 20 "Net-(ESP32-C3-Zero1-GP6)")
+	(net 21 "Net-(ESP32-C3-Zero1-GP10)")
+	(net 22 "Net-(ESP32-C3-Zero1-GP4)")
+	(net 23 "Net-(ESP32-C3-Zero1-GP19)")
+	(net 24 "Net-(ESP32-C3-Zero1-GP7)")
 	(net 25 "Net-(J16-Pin_4)")
 	(net 26 "Net-(J16-Pin_3)")
@@
 		(tags "connector JST XH vertical")
 		(property "Reference" "J13"
-			(at 2.5 -3.55 360)
+			(at 2.5 -3.55 0)
 			(layer "F.SilkS")
 			(hide yes)
@@
 		)
 		(property "Value" "BRL SENSE"
-			(at 2.5 4.6 360)
+			(at 2.5 4.6 0)
 			(layer "F.SilkS")
 			(effects
@@
 		)
 		(fp_text user "${REFERENCE}"
-			(at 2.5 2.7 360)
+			(at 2.5 2.7 0)
 			(layer "F.Fab")
 			(effects
@@
 			(layers "*.Cu" "*.Mask")
 			(remove_unused_layers no)
-			(net 22 "Net-(EC3Z1-GP4)")
+			(net 22 "Net-(ESP32-C3-Zero1-GP4)")
 			(pinfunction "Pin_3")
 			(pintype "passive")
@@
 		(tags "connector JST XH vertical")
 		(property "Reference" "J14"
-			(at 3.75 -3.55 360)
+			(at 3.75 -3.55 0)
 			(layer "F.SilkS")
 			(hide yes)
@@
 		)
 		(fp_text user "${REFERENCE}"
-			(at 3.652 2.55 360)
+			(at 3.652 2.55 0)
 			(layer "F.Fab")
 			(effects
@@
 		(tags "connector JST XH vertical")
 		(property "Reference" "J10"
-			(at 1.25 -3.55 360)
+			(at 1.25 -3.55 0)
 			(layer "F.SilkS")
 			(hide yes)
@@
 		)
 		(property "Value" "ENC BTN"
-			(at 1.25 -3.556 360)
+			(at 1.25 -3.556 0)
 			(layer "F.SilkS")
 			(effects
@@
 		)
 		(fp_text user "${REFERENCE}"
-			(at 1.25 2.7 360)
+			(at 1.25 2.7 0)
 			(layer "F.Fab")
 			(effects
@@
 			(layers "*.Cu" "*.Mask")
 			(remove_unused_layers no)
-			(net 21 "Net-(EC3Z1-GP10)")
+			(net 21 "Net-(ESP32-C3-Zero1-GP10)")
 			(pinfunction "Pin_2")
 			(pintype "passive")
@@
 		(tags "connector JST XH vertical")
 		(property "Reference" "J4"
-			(at 1.25 -3.55 360)
+			(at 1.25 -3.55 0)
 			(layer "F.SilkS")
 			(hide yes)
@@
 		)
 		(property "Value" "INT BTN"
-			(at 1.25 4.6 360)
+			(at 1.25 4.6 0)
 			(layer "F.SilkS")
 			(effects
@@
 		)
 		(fp_text user "${REFERENCE}"
-			(at 1.25 2.7 360)
+			(at 1.25 2.7 0)
 			(layer "F.Fab")
 			(effects
@@
 			(layers "*.Cu" "*.Mask")
 			(remove_unused_layers no)
-			(net 19 "Net-(EC3Z1-GP9)")
+			(net 19 "Net-(ESP32-C3-Zero1-GP9)")
 			(pinfunction "Pin_2")
 			(pintype "passive")
@@
 			(remove_unused_layers no)
 			(roundrect_rratio 0.1470588235)
-			(net 15 "Net-(EC3Z1-GP5)")
+			(net 15 "Net-(ESP32-C3-Zero1-GP5)")
 			(pinfunction "Pin_1")
 			(pintype "passive")
@@
 			(layers "*.Cu" "*.Mask")
 			(remove_unused_layers no)
-			(net 18 "Net-(EC3Z1-GP18)")
+			(net 18 "Net-(ESP32-C3-Zero1-GP18)")
 			(pinfunction "Pin_3")
 			(pintype "passive")
@@
 		(tags "connector JST XH vertical")
 		(property "Reference" "J7"
-			(at 1.25 -3.55 360)
+			(at 1.25 -3.55 0)
 			(layer "F.SilkS")
 			(hide yes)
@@
 		)
 		(property "Footprint" "Connector_JST:JST_XH_B2B-XH-A_1x02_P2.50mm_Vertical"
-			(at 0 0 360)
+			(at 0 0 0)
 			(layer "F.Fab")
 			(hide yes)
@@
 		)
 		(property "Datasheet" ""
-			(at 0 0 360)
+			(at 0 0 0)
 			(layer "F.Fab")
 			(hide yes)
@@
 		)
 		(property "Description" ""
-			(at 0 0 360)
+			(at 0 0 0)
 			(layer "F.Fab")
 			(hide yes)
@@
 		)
 		(fp_text user "${REFERENCE}"
-			(at 1.25 2.7 360)
+			(at 1.25 2.7 0)
 			(layer "F.Fab")
 			(effects
@@
 			(layers "*.Cu" "*.Mask")
 			(remove_unused_layers no)
-			(net 24 "Net-(EC3Z1-GP7)")
+			(net 24 "Net-(ESP32-C3-Zero1-GP7)")
 			(pinfunction "Pin_2")
 			(pintype "passive")
@@
 		(tags "connector JST XH vertical")
 		(property "Reference" "J8"
-			(at 1.25 -3.55 360)
+			(at 1.25 -3.55 0)
 			(layer "F.SilkS")
 			(hide yes)
@@
 		)
 		(property "Footprint" "Connector_JST:JST_XH_B2B-XH-A_1x02_P2.50mm_Vertical"
-			(at 0 0 360)
+			(at 0 0 0)
 			(layer "F.Fab")
 			(hide yes)
@@
 		)
 		(property "Datasheet" ""
-			(at 0 0 360)
+			(at 0 0 0)
 			(layer "F.Fab")
 			(hide yes)
@@
 		)
 		(property "Description" ""
-			(at 0 0 360)
+			(at 0 0 0)
 			(layer "F.Fab")
 			(hide yes)
@@
 		)
 		(fp_text user "${REFERENCE}"
-			(at 1.25 2.7 360)
+			(at 1.25 2.7 0)
 			(layer "F.Fab")
 			(effects
@@
 			(layers "*.Cu" "*.Mask")
 			(remove_unused_layers no)
-			(net 14 "Net-(EC3Z1-GP8)")
+			(net 14 "Net-(ESP32-C3-Zero1-GP8)")
 			(pinfunction "Pin_2")
 			(pintype "passive")
@@
 		(tags "THT DIP DIL PDIP 2.54mm 7.62mm 300mil Socket")
 		(property "Reference" "U1"
-			(at 3.81 -2.33 360)
+			(at 3.81 -2.33 0)
 			(layer "F.SilkS")
 			(hide yes)
@@
 		)
 		(property "Value" "74AHC125"
-			(at 3.81 17.57 360)
+			(at 3.81 17.57 0)
 			(layer "F.Fab")
 			(effects
@@
 		)
 		(property "Footprint" "Package_DIP:DIP-14_W7.62mm_Socket"
-			(at 0 0 360)
+			(at 0 0 0)
 			(layer "F.Fab")
 			(hide yes)
@@
 		)
 		(property "Datasheet" ""
-			(at 0 0 360)
+			(at 0 0 0)
 			(layer "F.Fab")
 			(hide yes)
@@
 		)
 		(property "Description" ""
-			(at 0 0 360)
+			(at 0 0 0)
 			(layer "F.Fab")
 			(hide yes)
@@
 		)
 		(fp_text user "${REFERENCE}"
-			(at 3.81 7.62 360)
+			(at 3.81 7.62 0)
 			(layer "F.Fab")
 			(effects
@@
 			(layers "*.Cu" "*.Mask")
 			(remove_unused_layers no)
-			(net 23 "Net-(EC3Z1-GP19)")
+			(net 23 "Net-(ESP32-C3-Zero1-GP19)")
 			(pinfunction "2A")
 			(pintype "input")
@@
 		(layer "F.Cu")
 		(at 90.225 92.16)
-		(property "Reference" "EC3Z1"
+		(property "Reference" "ESP32-C3-Zero1"
 			(at 0 -0.5 0)
 			(unlocked yes)
@@
 			(layers "*.Cu" "*.Mask")
 			(remove_unused_layers no)
-			(net 17 "Net-(EC3Z1-GP2)")
+			(net 17 "Net-(ESP32-C3-Zero1-GP2)")
 			(pinfunction "GP2")
 			(pintype "bidirectional")
@@
 			(layers "*.Cu" "*.Mask")
 			(remove_unused_layers no)
-			(net 16 "Net-(EC3Z1-GP3)")
+			(net 16 "Net-(ESP32-C3-Zero1-GP3)")
 			(pinfunction "GP3")
 			(pintype "bidirectional")
@@
 			(layers "*.Cu" "*.Mask")
 			(remove_unused_layers no)
-			(net 22 "Net-(EC3Z1-GP4)")
+			(net 22 "Net-(ESP32-C3-Zero1-GP4)")
 			(pinfunction "GP4")
 			(pintype "bidirectional")
@@
 			(layers "*.Cu" "*.Mask")
 			(remove_unused_layers no)
-			(net 15 "Net-(EC3Z1-GP5)")
+			(net 15 "Net-(ESP32-C3-Zero1-GP5)")
 			(pinfunction "GP5")
 			(pintype "bidirectional")
@@
 			(layers "*.Cu" "*.Mask")
 			(remove_unused_layers no)
-			(net 20 "Net-(EC3Z1-GP6)")
+			(net 20 "Net-(ESP32-C3-Zero1-GP6)")
 			(pinfunction "GP6")
 			(pintype "bidirectional")
@@
 			(layers "*.Cu" "*.Mask")
 			(remove_unused_layers no)
-			(net 24 "Net-(EC3Z1-GP7)")
+			(net 24 "Net-(ESP32-C3-Zero1-GP7)")
 			(pinfunction "GP7")
 			(pintype "bidirectional")
@@
 			(layers "*.Cu" "*.Mask")
 			(remove_unused_layers no)
-			(net 14 "Net-(EC3Z1-GP8)")
+			(net 14 "Net-(ESP32-C3-Zero1-GP8)")
 			(pinfunction "GP8")
 			(pintype "bidirectional")
@@
 			(layers "*.Cu" "*.Mask")
 			(remove_unused_layers no)
-			(net 19 "Net-(EC3Z1-GP9)")
+			(net 19 "Net-(ESP32-C3-Zero1-GP9)")
 			(pinfunction "GP9")
 			(pintype "bidirectional")
@@
 			(layers "*.Cu" "*.Mask")
 			(remove_unused_layers no)
-			(net 21 "Net-(EC3Z1-GP10)")
+			(net 21 "Net-(ESP32-C3-Zero1-GP10)")
 			(pinfunction "GP10")
 			(pintype "bidirectional")
@@
 			(layers "*.Cu" "*.Mask")
 			(remove_unused_layers no)
-			(net 18 "Net-(EC3Z1-GP18)")
+			(net 18 "Net-(ESP32-C3-Zero1-GP18)")
 			(pinfunction "GP18")
 			(pintype "bidirectional")
@@
 			(layers "*.Cu" "*.Mask")
 			(remove_unused_layers no)
-			(net 23 "Net-(EC3Z1-GP19)")
+			(net 23 "Net-(ESP32-C3-Zero1-GP19)")
 			(pinfunction "GP19")
 			(pintype "bidirectional")
@@
 		(tags "connector JST XH vertical")
 		(property "Reference" "J6"
-			(at 1.25 -3.55 360)
+			(at 1.25 -3.55 0)
 			(layer "F.SilkS")
 			(hide yes)
@@
 		)
 		(fp_text user "${REFERENCE}"
-			(at 1.25 2.7 360)
+			(at 1.25 2.7 0)
 			(layer "F.Fab")
 			(effects
@@
 			(layers "*.Cu" "*.Mask")
 			(remove_unused_layers no)
-			(net 20 "Net-(EC3Z1-GP6)")
+			(net 20 "Net-(ESP32-C3-Zero1-GP6)")
 			(pinfunction "Pin_2")
 			(pintype "passive")
@@
 			(layers "*.Cu" "*.Mask")
 			(remove_unused_layers no)
-			(net 17 "Net-(EC3Z1-GP2)")
+			(net 17 "Net-(ESP32-C3-Zero1-GP2)")
 			(pinfunction "Pin_2")
 			(pintype "passive")
@@
 			(layers "*.Cu" "*.Mask")
 			(remove_unused_layers no)
-			(net 16 "Net-(EC3Z1-GP3)")
+			(net 16 "Net-(ESP32-C3-Zero1-GP3)")
 			(pintype "passive")
 		)
