File: PCBs/KiCad/Pack Board/Pack Board/Pack Board.kicad_sch (KiCad schematic)
At the start: 13 parts, among them J1 BRL LEDS, J2 BODY LEDS, J3 TIP LED, J4 BAR, J5 DISP, U1 Teensy4.0_AudioShield_REVD, U2 74AHC125

Commit message: Wand Board Updates
Parts:
- added J10: SND OUT, Connector_JST:JST_XH_B2B-XH-A_1x02_P2.50mm_Vertical, symbol Connector_Generic:Conn_01x02
- added J11: SND IN R, Connector_JST:JST_XH_B2B-XH-A_1x02_P2.50mm_Vertical, symbol Connector_Generic:Conn_01x02
- added J12: SND IN L, Connector_JST:JST_XH_B2B-XH-A_1x02_P2.50mm_Vertical, symbol Connector_Generic:Conn_01x02
- added J13: BT MOSFET, Connector_JST:JST_XH_B3B-XH-A_1x03_P2.50mm_Vertical, symbol Connector_Generic:Conn_01x03
- added J14: VENT MOSFET, Connector_JST:JST_XH_B3B-XH-A_1x03_P2.50mm_Vertical, symbol Connector_Generic:Conn_01x03
- added J15: ROT ENC, Connector_JST:JST_XH_B3B-XH-A_1x03_P2.50mm_Vertical, symbol Connector_Generic:Conn_01x03
- added J16: ROT SW, Connector_JST:JST_XH_B2B-XH-A_1x02_P2.50mm_Vertical, symbol Connector_Generic:Conn_01x02
- added J17: ION SW, Connector_JST:JST_XH_B2B-XH-A_1x02_P2.50mm_Vertical, symbol Connector_Generic:Conn_01x02
- added J6: SERIAL, TerminalBlock_Phoenix:TerminalBlock_Phoenix_MKDS-1,5-2_1x02_P5.00mm_Horizontal, symbol Connector_Generic:Conn_01x02
- added J7: POW_IN, TerminalBlock_Phoenix:TerminalBlock_Phoenix_MKDS-1,5-2_1x02_P5.00mm_Horizontal, symbol Connector_Generic:Conn_01x02
- added J8: WAND PWR, TerminalBlock_Phoenix:TerminalBlock_Phoenix_MKDS-1,5-2_1x02_P5.00mm_Horizontal, symbol Connector_Generic:Conn_01x02
- added J9: AMP VOL, Connector_JST:JST_XH_B4B-XH-A_1x04_P2.50mm_Vertical, symbol Connector_Generic:Conn_01x04
- J1: value BRL LEDS -> VENT LIGHTS; footprint ProtonPackFootprints:JST_XH_B3B-XH-A_1x03_NeoPixelHeader -> Connector_JST:JST_XH_B3B-XH-A_1x03_P2.50mm_Vertical
- J2: value BODY LEDS -> PCELL LIGHTS; footprint ProtonPackFootprints:JST_XH_B3B-XH-A_1x03_NeoPixelHeader -> Connector_JST:JST_XH_B3B-XH-A_1x03_P2.50mm_Vertical
- J3: value TIP LED -> CYCLO LIGHTS; footprint ProtonPackFootprints:JST_XH_B3B-XH-A_1x03_NeoPixelHeader -> Connector_JST:JST_XH_B3B-XH-A_1x03_P2.50mm_Vertical
Connections:
- net SCL is gone; now on net GND: J4.4 (Pin_4), J5.4 (Pin_4), R5.1
- net SDA: now also U1.22 (18_A4_SDA0), J9.3 (Pin_3)
- net GND: now reaches J4.1 (Pin_1), J5.1 (Pin_1)
- net GND: now also C1.2, J1.1 (Pin_1), J2.1 (Pin_1), J3.1 (Pin_1), U1.1 (GND), U1.23 (19_A5_SCL0), U1.29 (GND), U2.10 (3OE), U2.13 (4OE), U2.4 (2OE), U2.7 (GND), J13.1 (Pin_1), J14.1 (Pin_1), J15.2 (Pin_2), J16.1 (Pin_1), J17.1 (Pin_1), J7.1 (Pin_1), J8.1 (Pin_1), J9.1 (Pin_1), J9.4 (Pin_4)
- net +3.3V: now reaches J4.2 (Pin_2), J5.2 (Pin_2), R4.2, R5.2
- net +3.3V: now also U1.28 (3V), J13.2 (Pin_2), J14.2 (Pin_2), J9.2 (Pin_2)
- net at U2.12 (4A): now also U1.18 (14_A0_TX3_SPDIF_OUT)
- net +5V: now reaches U2.14 (VCC)
- net +5V: now also C1.1, J1.2 (Pin_2), J2.2 (Pin_2), J3.2 (Pin_2), U1.30 (5V), J7.2 (Pin_2), J8.2 (Pin_2)
- net at U2.5 (2A): now also U1.21 (17_A3_TX4_SDA1)
- net at U2.9 (3A): now also U1.20 (16_A2_RX4_SCL1)
- net at U1.11 (9_OUT1C): now also J16.2 (Pin_2)
- net RX: now reaches U1.2 (0_RX1_CRX2_CS1)
- net RX: now also J6.2 (Pin_2)
- net at U1.26 (22_A8_CTX1): now also J17.2 (Pin_2)
- net TX: now reaches U1.3 (1_TX1_CTX2_MISO1)
- net TX: now also J6.1 (Pin_1)
- net at U1.31 (LINE_OUT_L): now also J10.2 (Pin_2)
- net at U1.32 (LINE_OUT_GND): now also J10.1 (Pin_1)
- net at U1.34 (LINE_IN_R): now also J11.2 (Pin_2)
- net at U1.35 (LINE_IN_L): now also J12.2 (Pin_2)
- net at U1.36 (LINE_IN_R_GND): now also J11.1 (Pin_1)
- net at U1.37 (LINE_IN_L_GND): now also J12.1 (Pin_1)
- net at U1.4 (2_OUT2): now also J15.1 (Pin_1)
- net at U1.5 (3_LRCLK2): now also J13.3 (Pin_3)
- net at U1.6 (4_BCLK2): now also J15.3 (Pin_3)
- net at U1.7 (5_IN2): now also J14.3 (Pin_3)
Other:
- moved on the sheet: U1

Commit message: Added motor output for wand rumble
Parts:
- added J18: i2c Extend, Connector_JST:JST_XH_B4B-XH-A_1x04_P2.50mm_Vertical, symbol Connector_Generic:Conn_01x04
Connections:
- net +3.3V: now also J18.2 (Pin_2)
- net GND: now also J18.1 (Pin_1), J18.4 (Pin_4)
- net SDA: now also J18.3 (Pin_3)
- no-connect marks 3 -> 23
Changed lines of the file:
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@@
   (junction (at 116.84 25.4) (diameter 0) (color 0 0 0 0)
   )
+  (junction (at 217.17 140.97) (diameter 0) (color 0 0 0 0)
+  )
   (junction (at 207.01 25.4) (diameter 0) (color 0 0 0 0)
   )
@@
   (junction (at 220.98 127) (diameter 0) (color 0 0 0 0)
   )
+  (junction (at 214.63 138.43) (diameter 0) (color 0 0 0 0)
+  )
   (junction (at 38.1 97.79) (diameter 0) (color 0 0 0 0)
   )
@@
   (junction (at 175.26 30.48) (diameter 0) (color 0 0 0 0)
   )
+  (junction (at 212.09 135.89) (diameter 0) (color 0 0 0 0)
+  )
   (junction (at 123.19 25.4) (diameter 0) (color 0 0 0 0)
   )
   (junction (at 93.98 105.41) (diameter 0) (color 0 0 0 0)
   )
+  (junction (at 220.98 143.51) (diameter 0) (color 0 0 0 0)
+  )
   (junction (at 160.02 30.48) (diameter 0) (color 0 0 0 0)
   )
@@
   )
   (no_connect (at 55.88 95.25))
+  (no_connect (at 115.57 91.44))
+  (no_connect (at 115.57 83.82))
+  (no_connect (at 171.45 66.04))
+  (no_connect (at 171.45 80.01))
+  (no_connect (at 171.45 63.5))
+  (no_connect (at 171.45 129.54))
+  (no_connect (at 115.57 116.84))
+  (no_connect (at 115.57 132.08))
+  (no_connect (at 171.45 77.47))
+  (no_connect (at 115.57 102.87))
+  (no_connect (at 115.57 81.28))
+  (no_connect (at 115.57 93.98))
+  (no_connect (at 171.45 102.87))
+  (no_connect (at 115.57 105.41))
+  (no_connect (at 115.57 86.36))
   (no_connect (at 50.8 95.25))
+  (no_connect (at 171.45 68.58))
   (no_connect (at 45.72 95.25))
+  (no_connect (at 115.57 96.52))
+  (no_connect (at 171.45 74.93))
+  (no_connect (at 115.57 129.54))
+  (no_connect (at 115.57 111.76))
   (wire (pts (xy 93.98 27.94) (xy 93.98 105.41))
     (stroke (width 0) (type default))
@@
     (stroke (width 0) (type default))
   )
+  (wire (pts (xy 224.79 151.13) (xy 212.09 151.13))
+    (stroke (width 0) (type default))
+  )
   (wire (pts (xy 45.72 130.81) (xy 46.99 130.81))
     (stroke (width 0) (type default))
@@
     (stroke (width 0) (type default))
   )
+  (wire (pts (xy 214.63 153.67) (xy 214.63 138.43))
+    (stroke (width 0) (type default))
+  )
   (wire (pts (xy 113.03 137.16) (xy 208.28 137.16))
     (stroke (width 0) (type default))
@@
     (stroke (width 0) (type default))
   )
+  (wire (pts (xy 220.98 158.75) (xy 220.98 143.51))
+    (stroke (width 0) (type default))
+  )
   (wire (pts (xy 68.58 95.25) (xy 68.58 121.92))
     (stroke (width 0) (type default))
@@
     (stroke (width 0) (type default))
   )
+  (wire (pts (xy 224.79 153.67) (xy 214.63 153.67))
+    (stroke (width 0) (type default))
+  )
+  (wire (pts (xy 212.09 151.13) (xy 212.09 135.89))
+    (stroke (width 0) (type default))
+  )
   (wire (pts (xy 30.48 25.4) (xy 30.48 57.15))
     (stroke (width 0) (type default))
@@
     (stroke (width 0) (type default))
   )
+  (wire (pts (xy 217.17 156.21) (xy 217.17 140.97))
+    (stroke (width 0) (type default))
+  )
   (wire (pts (xy 93.98 146.05) (xy 93.98 133.35))
     (stroke (width 0) (type default))
@@
     (stroke (width 0) (type default))
   )
+  (wire (pts (xy 224.79 156.21) (xy 217.17 156.21))
+    (stroke (width 0) (type default))
+  )
   (wire (pts (xy 160.02 30.48) (xy 175.26 30.48))
     (stroke (width 0) (type default))
   )
   (wire (pts (xy 171.45 107.95) (xy 184.15 107.95))
+    (stroke (width 0) (type default))
+  )
+  (wire (pts (xy 224.79 158.75) (xy 220.98 158.75))
     (stroke (width 0) (type default))
   )
@@
         )
       )
+    )
+  )
+  (symbol (lib_id "Connector_Generic:Conn_01x04") (at 229.87 153.67 0) (unit 1)
+    (in_bom yes) (on_board yes) (dnp no) (fields_autoplaced)
+    (property "Reference" "J18" (at 232.41 153.67 0)
+      (effects (font (size 1.27 1.27)) (justify left))
+    )
+    (property "Value" "i2c Extend" (at 232.41 156.21 0)
+      (effects (font (size 1.27 1.27)) (justify left))
+    )
+    (property "Footprint" "Connector_JST:JST_XH_B4B-XH-A_1x04_P2.50mm_Vertical" (at 229.87 153.67 0)
+      (effects (font (size 1.27 1.27)) hide)
+    )
+    (property "Datasheet" "~" (at 229.87 153.67 0)
+      (effects (font (size 1.27 1.27)) hide)
+    )
+    (pin "1")
+    (pin "2")
+    (pin "3")
+    (pin "4")
+    (instances
+      (project "Pack Board"
+        (path "/01028740-8ea4-4743-b5bb-e9232ee12845"
+          (reference "J18") (unit 1)
+        )
+      )
+      (project "Wand Board"
+        (path "/1c8798cf-59eb-4db0-a440-e8dd7a851253"
+          (reference "J15") (unit 1)
+        )
+      )

Commit message: Added additional i2c output to wand board for optional driver
Parts:
- removed J4: BAR, Connector_JST:JST_XH_B4B-XH-A_1x04_P2.50mm_Vertical, symbol Connector_Generic:Conn_01x04
- removed J5: DISP, Connector_JST:JST_XH_B4B-XH-A_1x04_P2.50mm_Vertical, symbol Connector_Generic:Conn_01x04
- U1: symbol teensy:Teensy4.0_AudioShield_REVD -> teensy:Teensy4.0_AudioShield_REVD_Teensy_and_AudioInOutOnly
Connections:
- no-connect marks 23 -> 15
Changed lines of the file:
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@@
   (junction (at 86.36 135.89) (diameter 0) (color 0 0 0 0)
   )
-  (junction (at 212.09 100.33) (diameter 0) (color 0 0 0 0)
-  )
   (junction (at 86.36 25.4) (diameter 0) (color 0 0 0 0)
   )
   (junction (at 172.72 27.94) (diameter 0) (color 0 0 0 0)
   )
-  (junction (at 217.17 124.46) (diameter 0) (color 0 0 0 0)
-  )
   (junction (at 86.36 123.19) (diameter 0) (color 0 0 0 0)
   )
@@
   (junction (at 86.36 105.41) (diameter 0) (color 0 0 0 0)
   )
-  (junction (at 214.63 102.87) (diameter 0) (color 0 0 0 0)
-  )
   (junction (at 63.5 25.4) (diameter 0) (color 0 0 0 0)
   )
@@
   (junction (at 73.66 148.59) (diameter 0) (color 0 0 0 0)
   )
-  (junction (at 220.98 127) (diameter 0) (color 0 0 0 0)
-  )
   (junction (at 214.63 138.43) (diameter 0) (color 0 0 0 0)
   )
@@
   )
   (junction (at 199.39 102.87) (diameter 0) (color 0 0 0 0)
-  )
-  (junction (at 212.09 119.38) (diameter 0) (color 0 0 0 0)
-  )
-  (junction (at 214.63 121.92) (diameter 0) (color 0 0 0 0)
   )
   (junction (at 199.39 124.46) (diameter 0) (color 0 0 0 0)
@@
   (no_connect (at 115.57 91.44))
   (no_connect (at 115.57 83.82))
-  (no_connect (at 171.45 66.04))
-  (no_connect (at 171.45 80.01))
-  (no_connect (at 171.45 63.5))
   (no_connect (at 171.45 129.54))
   (no_connect (at 115.57 116.84))
   (no_connect (at 115.57 132.08))
-  (no_connect (at 171.45 77.47))
-  (no_connect (at 115.57 102.87))
   (no_connect (at 115.57 81.28))
   (no_connect (at 115.57 93.98))
   (no_connect (at 171.45 102.87))
-  (no_connect (at 115.57 105.41))
   (no_connect (at 115.57 86.36))
   (no_connect (at 50.8 95.25))
-  (no_connect (at 171.45 68.58))
   (no_connect (at 45.72 95.25))
   (no_connect (at 115.57 96.52))
-  (no_connect (at 171.45 74.93))
   (no_connect (at 115.57 129.54))
   (no_connect (at 115.57 111.76))
@@
     (stroke (width 0) (type default))
   )
-  (wire (pts (xy 214.63 138.43) (xy 214.63 121.92))
-    (stroke (width 0) (type default))
-  )
   (wire (pts (xy 100.33 154.94) (xy 124.46 154.94))
     (stroke (width 0) (type default))
@@
     (stroke (width 0) (type default))
   )
-  (wire (pts (xy 220.98 107.95) (xy 220.98 127))
-    (stroke (width 0) (type default))
-  )
   (wire (pts (xy 207.01 82.55) (xy 207.01 91.44))
     (stroke (width 0) (type default))
@@
     (stroke (width 0) (type default))
   )
-  (wire (pts (xy 224.79 121.92) (xy 214.63 121.92))
-    (stroke (width 0) (type default))
-  )
   (wire (pts (xy 95.25 149.86) (xy 55.88 149.86))
     (stroke (width 0) (type default))
@@
     (stroke (width 0) (type default))
   )
-  (wire (pts (xy 217.17 124.46) (xy 224.79 124.46))
-    (stroke (width 0) (type default))
-  )
   (wire (pts (xy 38.1 97.79) (xy 30.48 97.79))
     (stroke (width 0) (type default))
   )
-  (wire (pts (xy 217.17 105.41) (xy 217.17 124.46))
-    (stroke (width 0) (type default))
-  )
   (wire (pts (xy 208.28 137.16) (xy 208.28 127))
     (stroke (width 0) (type default))
@@
     (stroke (width 0) (type default))
   )
-  (wire (pts (xy 214.63 121.92) (xy 214.63 102.87))
+  (wire (pts (xy 214.63 102.87) (xy 214.63 138.43))
     (stroke (width 0) (type default))
   )
@@
     (stroke (width 0) (type default))
   )
-  (wire (pts (xy 212.09 135.89) (xy 212.09 119.38))
-    (stroke (width 0) (type default))
-  )
-  (wire (pts (xy 212.09 119.38) (xy 212.09 100.33))
+  (wire (pts (xy 212.09 100.33) (xy 212.09 135.89))
     (stroke (width 0) (type default))
   )
@@
     (stroke (width 0) (type default))
   )
-  (wire (pts (xy 224.79 105.41) (xy 217.17 105.41))
-    (stroke (width 0) (type default))
-  )
   (wire (pts (xy 86.36 25.4) (xy 86.36 105.41))
     (stroke (width 0) (type default))
   )
-  (wire (pts (xy 212.09 100.33) (xy 224.79 100.33))
-    (stroke (width 0) (type default))
-  )
   (wire (pts (xy 172.72 121.92) (xy 171.45 121.92))
     (stroke (width 0) (type default))
@@
     (stroke (width 0) (type default))
   )
-  (wire (pts (xy 214.63 102.87) (xy 224.79 102.87))
-    (stroke (width 0) (type default))
-  )
   (wire (pts (xy 116.84 25.4) (xy 123.19 25.4))
     (stroke (width 0) (type default))
   )
-  (wire (pts (xy 220.98 127) (xy 224.79 127))
-    (stroke (width 0) (type default))
-  )
   (wire (pts (xy 199.39 118.11) (xy 199.39 124.46))
     (stroke (width 0) (type default))
@@
     (stroke (width 0) (type default))
   )
-  (wire (pts (xy 224.79 107.95) (xy 220.98 107.95))
-    (stroke (width 0) (type default))
-  )
   (wire (pts (xy 107.95 53.34) (xy 107.95 68.58))
     (stroke (width 0) (type default))
@@
   )
   (wire (pts (xy 184.15 107.95) (xy 184.15 148.59))
-    (stroke (width 0) (type default))
-  )
-  (wire (pts (xy 224.79 119.38) (xy 212.09 119.38))
     (stroke (width 0) (type default))
   )
@@
         (path "/1c8798cf-59eb-4db0-a440-e8dd7a851253"
           (reference "J5") (unit 1)
-        )
-      )
-    )
-  )
-  (symbol (lib_id "Connector_Generic:Conn_01x04") (at 229.87 102.87 0) (unit 1)
-    (in_bom yes) (on_board yes) (dnp no) (fields_autoplaced)
-    (property "Reference" "J4" (at 232.41 102.87 0)
-      (effects (font (size 1.27 1.27)) (justify left))
-    )
-    (property "Value" "BAR" (at 232.41 105.41 0)
-      (effects (font (size 1.27 1.27)) (justify left))
-    )
-    (property "Footprint" "Connector_JST:JST_XH_B4B-XH-A_1x04_P2.50mm_Vertical" (at 229.87 102.87 0)
-      (effects (font (size 1.27 1.27)) hide)
-    )
-    (property "Datasheet" "~" (at 229.87 102.87 0)
-      (effects (font (size 1.27 1.27)) hide)
-    )
-    (pin "1")
-    (pin "2")
-    (pin "3")
-    (pin "4")
-    (instances
-      (project "Pack Board"
-        (path "/01028740-8ea4-4743-b5bb-e9232ee12845"
-          (reference "J4") (unit 1)
-        )
-      )
-      (project "Wand Board"
-        (path "/1c8798cf-59eb-4db0-a440-e8dd7a851253"
-          (reference "J14") (unit 1)
         )
       )
@@
     )
   )
-  (symbol (lib_id "teensy:Teensy4.0_AudioShield_REVD") (at 143.51 97.79 0) (unit 1)
+  (symbol (lib_id "teensy:Teensy4.0_AudioShield_REVD_Teensy_and_AudioInOutOnly") (at 143.51 97.79 0) (unit 1)
     (in_bom yes) (on_board yes) (dnp no) (fields_autoplaced)
     (property "Reference" "U1" (at 143.51 55.88 0)
@@
     (pin "13")
     (pin "14")
-    (pin "15")
-    (pin "16")
     (pin "17")
     (pin "18")
@@
     (pin "36")
     (pin "37")
-    (pin "38")
-    (pin "39")
-    (pin "40")
-    (pin "41")
-    (pin "42")
-    (pin "43")
     (pin "5")
     (pin "6")
@@
     (pin "8")
     (pin "9")
+    (pin "45")
+    (pin "46")
     (pin "1")
     (pin "2")
@@
         )
       )
-      (project "Wand Board"
-        (path "/1c8798cf-59eb-4db0-a440-e8dd7a851253"
-          (reference "J15") (unit 1)
-        )
-      )
-    )
-  )
-  (symbol (lib_id "Connector_Generic:Conn_01x04") (at 229.87 121.92 0) (unit 1)
-    (in_bom yes) (on_board yes) (dnp no) (fields_autoplaced)
-    (property "Reference" "J5" (at 232.41 121.92 0)
-      (effects (font (size 1.27 1.27)) (justify left))
-    )
-    (property "Value" "DISP" (at 232.41 124.46 0)
-      (effects (font (size 1.27 1.27)) (justify left))
-    )
-    (property "Footprint" "Connector_JST:JST_XH_B4B-XH-A_1x04_P2.50mm_Vertical" (at 229.87 121.92 0)
-      (effects (font (size 1.27 1.27)) hide)
-    )
-    (property "Datasheet" "~" (at 229.87 121.92 0)
-      (effects (font (size 1.27 1.27)) hide)
-    )
-    (pin "1")
-    (pin "2")
-    (pin "3")
-    (pin "4")
-    (instances
-      (project "Pack Board"
-        (path "/01028740-8ea4-4743-b5bb-e9232ee12845"
-          (reference "J5") (unit 1)
-        )
-      )

Commit message: Pack Board 2.0
Connections:
- net LINE_IN_R_GND: now reaches J11.1 (Pin_1), U1.36 (LINE_IN_R_GND)
- net LINE_IN_R: now reaches J11.2 (Pin_2), U1.34 (LINE_IN_R)
- net LINE_IN_L_GND: now reaches J12.1 (Pin_1), U1.37 (LINE_IN_L_GND)
- net LINE_IN_L: now reaches J12.2 (Pin_2), U1.35 (LINE_IN_L)
- net at U2.12 (4A): now also U1.21 (17_A3_TX4_SDA1); no longer U1.18 (14_A0_TX3_SPDIF_OUT)
- net at U2.5 (2A): now also U1.18 (14_A0_TX3_SPDIF_OUT); no longer U1.21 (17_A3_TX4_SDA1)
- net at U1.11 (9_OUT1C): now also J13.3 (Pin_3); no longer J16.2 (Pin_2)
- net LINE_OUT_L: now reaches J10.2 (Pin_2), U1.31 (LINE_OUT_L)
- net LINE_OUT_L: now also U1.46 (NCA)
- net LINE_OUT_GND: now reaches J10.1 (Pin_1), U1.32 (LINE_OUT_GND)
- net at U1.4 (2_OUT2): now also J16.2 (Pin_2); no longer J15.1 (Pin_1)
- net at U1.5 (3_LRCLK2): now also J15.3 (Pin_3); no longer J13.3 (Pin_3)
- net at U1.6 (4_BCLK2): now also J15.1 (Pin_1); no longer J15.3 (Pin_3)
Other:
- moved on the sheet: R1, R3

Commit message: Pack PCB tweaks for 5V triggered FET/Relays, consolidating LED pins, and breaking out newly freed  I/O pin.  Re-jigged board layout and fixed some dimensions.
Parts:
- removed J2: PCELL LIGHTS, Connector_JST:JST_XH_B3B-XH-A_1x03_P2.50mm_Vertical, symbol Connector_Generic:Conn_01x03
- removed R1, R3: 220, Resistor_THT:R_Axial_DIN0207_L6.3mm_D2.5mm_P7.62mm_Horizontal, symbol Device:R
- added J4: PCELL LIGHTS, ProtonPackFootprints:JST_XH_B4B-XH-A_1x04_NeoPixelHeader, symbol Connector_Generic:Conn_01x04
- added J5: SPARE IO, ProtonPackFootprints:JST_XH_B2B-XH-A_1x02_P2.50mm_Vertical, symbol Connector_Generic:Conn_01x02
- J1: value VENT LIGHTS -> VENT SMOKE; footprint Connector_JST:JST_XH_B3B-XH-A_1x03_P2.50mm_Vertical -> ProtonPackFootprints:JST_XH_B3B-XH-A_1x03_MosRelay
- J10, J11, J12: footprint Connector_JST:JST_XH_B2B-XH-A_1x02_P2.50mm_Vertical -> ProtonPackFootprints:JST_XH_B2B-XH-A_1x02_AudioHeader
- J13: value BT MOSFET -> BT AUDIO; footprint Connector_JST:JST_XH_B3B-XH-A_1x03_P2.50mm_Vertical -> ProtonPackFootprints:JST_XH_B3B-XH-A_1x03_MosRelay
- J14: value VENT MOSFET -> VENT FAN; footprint Connector_JST:JST_XH_B3B-XH-A_1x03_P2.50mm_Vertical -> ProtonPackFootprints:JST_XH_B3B-XH-A_1x03_MosRelay
- J15: footprint Connector_JST:JST_XH_B3B-XH-A_1x03_P2.50mm_Vertical -> ProtonPackFootprints:JST_XH_B3B-XH-A_1x03_RotEncoder
- J16, J17: footprint Connector_JST:JST_XH_B2B-XH-A_1x02_P2.50mm_Vertical -> ProtonPackFootprints:JST_XH_B2B-XH-A_1x02_P2.50mm_Vertical
- J18, J9: footprint Connector_JST:JST_XH_B4B-XH-A_1x04_P2.50mm_Vertical -> ProtonPackFootprints:JST_XH_B4B-XH-A_1x04_i2cHeader
- J3: footprint Connector_JST:JST_XH_B3B-XH-A_1x03_P2.50mm_Vertical -> ProtonPackFootprints:JST_XH_B3B-XH-A_1x03_NeoPixelHeader
- J6, J7, J8: footprint TerminalBlock_Phoenix:TerminalBlock_Phoenix_MKDS-1,5-2_1x02_P5.00mm_Horizontal -> ProtonPackFootprints:TerminalBlock_Phoenix_MKDS-1,5-2_1x02_P5.00mm_Horizontal
- R2, R4, R5: footprint Resistor_THT:R_Axial_DIN0207_L6.3mm_D2.5mm_P7.62mm_Horizontal -> ProtonPackFootprints:R_Axial_DIN0207_L6.3mm_D2.5mm_P7.62mm_Horizontal
- U1: footprint Teensy:4.0audioshield -> ProtonPackFootprints:Teensy Audioshield Rev D
Connections:
- net +3.3V: no longer J13.2 (Pin_2), J14.2 (Pin_2)
- net +5V: now also J13.2 (Pin_2), J14.2 (Pin_2), J4.2 (Pin_2)
- net GND: now also U2.1 (1OE), J4.1 (Pin_1), J5.1 (Pin_1); no longer J18.4 (Pin_4), J9.4 (Pin_4), R5.1, U1.23 (19_A5_SCL0)
- net RX: now also U1.3 (1_TX1_CTX2_MISO1); no longer U1.2 (0_RX1_CRX2_CS1)
- net TX: now also U1.2 (0_RX1_CRX2_CS1); no longer U1.3 (1_TX1_CTX2_MISO1)
- net at J17.2 (Pin_2): now also U1.18 (14_A0_TX3_SPDIF_OUT); no longer U1.26 (22_A8_CTX1)
- net CYCLO_LED_IN: now reaches J3.3 (Pin_3)
- net CYCLO_LED_IN: now also J4.4 (Pin_4)
- net at U2.11 (4Y): now also J1.3 (Pin_3)
- net at U2.12 (4A): now also U1.11 (9_OUT1C); no longer U1.21 (17_A3_TX4_SDA1)
- net at U2.2 (1A): now also U1.7 (5_IN2)
- net at U2.3 (1Y): now also J14.3 (Pin_3)
- net at U2.5 (2A): now also U1.21 (17_A3_TX4_SDA1); no longer U1.18 (14_A0_TX3_SPDIF_OUT)
- net at U2.6 (2Y): now also J13.3 (Pin_3)
- net LED_IN: now reaches R2.2, U2.8 (3Y)
- net at U1.5 (3_LRCLK2): now also J15.1 (Pin_1); no longer J15.3 (Pin_3)
- net at U1.6 (4_BCLK2): now also J15.3 (Pin_3); no longer J15.1 (Pin_1)
- net PCELL_LED_IN: now reaches R2.1
- net PCELL_LED_IN: now also J4.3 (Pin_3)
- new net: J5.2 (Pin_2), U1.26 (22_A8_CTX1)
- new net SCL: J18.4 (Pin_4), J9.4 (Pin_4), R5.1, U1.23 (19_A5_SCL0)
- no-connect marks 15 -> 12
Other:
- moved on the sheet: J13, R2
